File: ch340_module.kicad_pcb (KiCad board)
At the start: 2 copper layers, 13 x 37 mm, 11 parts, among them J1 UART Device, J2 USB, U1 CH340K, U2 LTV-817S, U3 LTV-817S

Commit message: readme
Parts:
- C1, C2: value 0.1nF -> 0.1uF
- moved R1 58.0 mm to (90.2, 62.8), turned to -90 degrees
- moved U3 55.8 mm to (97.5, 62.5), turned to 0 degrees
- moved R2 54.8 mm to (105.2, 62.4), turned to 90 degrees
- moved J2 53.4 mm to (118.0, 65.5), turned to 90 degrees
- moved U1 53.1 mm to (110.9, 64.0), turned to 180 degrees
- moved J1 52.0 mm to (87.2, 69.3), turned to 180 degrees
- moved R4 52.0 mm to (90.2, 67.8), turned to -90 degrees
- moved U2 47.6 mm to (97.5, 68.5), turned to 180 degrees
- moved C2 46.9 mm to (105.2, 68.0), turned to -90 degrees
- moved C1 45.8 mm to (112.8, 69.5), turned to 0 degrees
- moved R3 44.9 mm to (108.5, 69.5), turned to 180 degrees
Connections:
- net Net-(J1-Pin_2) renamed /RX
- net Net-(J1-Pin_3) renamed /TX
- C2 pad 1: VCC -> GND2
Routing:
- net VCC: track 38.1 -> 27.5 mm
- net GND2: track 0.00 -> 1.62 mm
- net /RX: track 5.67 -> 6.92 mm
Other:
- board size 13 x 37 mm -> 37 x 13 mm
